File: hardware/puck-revA/puck-revA.kicad_sch (KiCad schematic)
At the start: 27 parts, among them J1 USB-C 16P, J2 UART, J3 EXP (DNP on the product), SW1 BOOT, SW2 RESET, SW3 USER, U1 ESP32-S3-WROOM-1-N16, U2 AP2112K-3.3, U3 74AHCT1G125, U4 USBLC6-2SC6, U5 ambient light, DNP

Commit message: hardware(puck): the library tables exist, and they found two real faults
Launching the KiCad GUI once writes the global symbol and footprint tables, and
ERC stopped complaining about missing libraries and started complaining about the
design. 49 warnings became 7, and the 7 were worth having.

U1 carried RF_Module:ESP32-S2-WROOM -- an S2 footprint on an S3 module, and one
that does not exist in the library either. It is ESP32-S3-WROOM-1 now.

The LEDs pointed at a PLCC6 land in a library called LED. SK6812-RGBW is PLCC4 in
LED_SMD: the W is a fourth die, not a fifth pin, so the part is still VDD/DOUT/
VSS/DIN and the WS2812B symbol is right for it after all. Nothing needed drawing.

The third fault was the interesting one, and ERC called it lib_symbol_mismatch,
which sounds cosmetic. A derived symbol's parent supplies geometry and nothing
else, but embed() was taking the parent's PROPERTIES too -- so the embedded
AP2112K-3.3 carried Value "AP2204K-1.5", a 150 mA regulator standing in for a 600
mA one, with a datasheet and a description to match. A wrong value on its way to
a BOM, wearing the clothes of a formatting warning. The child's properties are
overlaid on the parent's geometry now, and the same fix covers 74AHCT1G125 and
USBLC6-2SC6.

Every part has a real footprint from the stock libraries, the four that were left
blank included: the USB-C is a GCT USB4105, the buttons are side-actuated SKQG,
the headers are ordinary 2.54 mm verticals.

Now: 29 symbols, 22 nets, 0 wrong against PARTS, and ERC clean -- zero
violations. The ambient light sensor is still a stand-in (KiCad 10 ships no
VEML7700) and the README says so where the part is named, because a placeholder
that stops being visible is how it becomes the decision.

Co-Authored-By: Claude Opus 5 (1M context) <noreply@anthropic.com>
Parts:
- D1, D2, D3: footprint LED:LED_SK6812_PLCC6_5.0x5.0mm -> LED_SMD:LED_SK6812_PLCC4_5.0x5.0mm_P3.2mm
- J1: footprint (none) -> Connector_USB:USB_C_Receptacle_GCT_USB4105-xx-A_16P_TopMnt_Horizontal
- J2: footprint (none) -> Connector_PinHeader_2.54mm:PinHeader_1x04_P2.54mm_Vertical
- J3: footprint (none) -> Connector_PinHeader_2.54mm:PinHeader_1x06_P2.54mm_Vertical
- SW1, SW2, SW3: footprint (none) -> Button_Switch_SMD:SW_SPST_SKQG_WithoutStem
- U1: footprint RF_Module:ESP32-S2-WROOM -> RF_Module:ESP32-S3-WROOM-1
- U5: footprint (none) -> OptoDevice:Lite-On_LTR-303ALS-01
Changed lines of the file:
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@@
 			)
 		)
-		(property "Footprint" "RF_Module:ESP32-S2-WROOM"
+		(property "Footprint" "RF_Module:ESP32-S3-WROOM-1"
 			(at 83.82 81.98 0)
 			(effects
@@
 		(instances
 			(project "puck-revA"
-				(path "/5d319f43-1749-4bb5-87ad-5a3caec3474c"
+				(path "/95006bc4-82f3-4f47-9447-57085013e108"
 					(reference "U1")
 					(unit 1)
@@
 		(instances
 			(project "puck-revA"
-				(path "/5d319f43-1749-4bb5-87ad-5a3caec3474c"
+				(path "/95006bc4-82f3-4f47-9447-57085013e108"
 					(reference "U2")
 					(unit 1)
@@
 		(instances
 			(project "puck-revA"
-				(path "/5d319f43-1749-4bb5-87ad-5a3caec3474c"
+				(path "/95006bc4-82f3-4f47-9447-57085013e108"
 					(reference "U3")
 					(unit 1)
@@
 		(instances
 			(project "puck-revA"
-				(path "/5d319f43-1749-4bb5-87ad-5a3caec3474c"
+				(path "/95006bc4-82f3-4f47-9447-57085013e108"
 					(reference "U4")
 					(unit 1)
@@
 			)
 		)
-		(property "Footprint" ""
+		(property "Footprint" "OptoDevice:Lite-On_LTR-303ALS-01"
 			(at 375.92 64.20 0)
 			(effects
@@
 		(instances
 			(project "puck-revA"
-				(path "/5d319f43-1749-4bb5-87ad-5a3caec3474c"
+				(path "/95006bc4-82f3-4f47-9447-57085013e108"
 					(reference "U5")
 					(unit 1)
@@
 			)
 		)
-		(property "Footprint" ""
+		(property "Footprint" "Connector_USB:USB_C_Receptacle_GCT_USB4105-xx-A_16P_TopMnt_Horizontal"
 			(at 182.88 71.82 0)
 			(effects
@@
 		(instances
 			(project "puck-revA"
-				(path "/5d319f43-1749-4bb5-87ad-5a3caec3474c"
+				(path "/95006bc4-82f3-4f47-9447-57085013e108"
 					(reference "J1")
 					(unit 1)
@@
 			)
 		)
-		(property "Footprint" ""
+		(property "Footprint" "Connector_PinHeader_2.54mm:PinHeader_1x04_P2.54mm_Vertical"
 			(at 485.14 170.88 0)
 			(effects
@@
 		(instances
 			(project "puck-revA"
-				(path "/5d319f43-1749-4bb5-87ad-5a3caec3474c"
+				(path "/95006bc4-82f3-4f47-9447-57085013e108"
 					(reference "J2")
 					(unit 1)
@@
 			)
 		)
-		(property "Footprint" ""
+		(property "Footprint" "Connector_PinHeader_2.54mm:PinHeader_1x06_P2.54mm_Vertical"
 			(at 325.12 173.42 0)
 			(effects
@@
 		(instances
 			(project "puck-revA"
-				(path "/5d319f43-1749-4bb5-87ad-5a3caec3474c"
+				(path "/95006bc4-82f3-4f47-9447-57085013e108"
 					(reference "J3")
 					(unit 1)
@@
 			)
 		)
-		(property "Footprint" "LED:LED_SK6812_PLCC6_5.0x5.0mm"
+		(property "Footprint" "LED_SMD:LED_SK6812_PLCC4_5.0x5.0mm_P3.2mm"
 			(at 467.36 61.66 0)
 			(effects
@@
 		(instances
 			(project "puck-revA"
-				(path "/5d319f43-1749-4bb5-87ad-5a3caec3474c"
+				(path "/95006bc4-82f3-4f47-9447-57085013e108"
 					(reference "D1")
 					(unit 1)
@@
 			)
 		)
-		(property "Footprint" "LED:LED_SK6812_PLCC6_5.0x5.0mm"
+		(property "Footprint" "LED_SMD:LED_SK6812_PLCC4_5.0x5.0mm_P3.2mm"
 			(at 76.20 173.42 0)
 			(effects
@@
 		(instances
 			(project "puck-revA"
-				(path "/5d319f43-1749-4bb5-87ad-5a3caec3474c"
+				(path "/95006bc4-82f3-4f47-9447-57085013e108"
 					(reference "D2")
 					(unit 1)
@@
 			)
 		)
-		(property "Footprint" "LED:LED_SK6812_PLCC6_5.0x5.0mm"
+		(property "Footprint" "LED_SMD:LED_SK6812_PLCC4_5.0x5.0mm_P3.2mm"
 			(at 165.10 173.42 0)
 			(effects
@@
 		(instances
 			(project "puck-revA"
-				(path "/5d319f43-1749-4bb5-87ad-5a3caec3474c"
+				(path "/95006bc4-82f3-4f47-9447-57085013e108"
 					(reference "D3")
 					(unit 1)
@@
 			)
 		)
-		(property "Footprint" ""
+		(property "Footprint" "Button_Switch_SMD:SW_SPST_SKQG_WithoutStem"
 			(at 505.46 300.42 0)
 			(effects
@@
 		(instances
 			(project "puck-revA"
-				(path "/5d319f43-1749-4bb5-87ad-5a3caec3474c"
+				(path "/95006bc4-82f3-4f47-9447-57085013e108"
 					(reference "SW1")
 					(unit 1)
@@
 			)
 		)
-		(property "Footprint" ""
+		(property "Footprint" "Button_Switch_SMD:SW_SPST_SKQG_WithoutStem"
 			(at 73.66 363.92 0)
 			(effects
@@
 		(instances
 			(project "puck-revA"
-				(path "/5d319f43-1749-4bb5-87ad-5a3caec3474c"
+				(path "/95006bc4-82f3-4f47-9447-57085013e108"
 					(reference "SW2")
 					(unit 1)
@@
 			)
 		)
-		(property "Footprint" ""
+		(property "Footprint" "Button_Switch_SMD:SW_SPST_SKQG_WithoutStem"
 			(at 157.48 363.92 0)
 			(effects
@@
 		(instances
 			(project "puck-revA"
-				(path "/5d319f43-1749-4bb5-87ad-5a3caec3474c"
+				(path "/95006bc4-82f3-4f47-9447-57085013e108"
 					(reference "SW3")
 					(unit 1)
@@
 		(instances
 			(project "puck-revA"
-				(path "/5d319f43-1749-4bb5-87ad-5a3caec3474c"
+				(path "/95006bc4-82f3-4f47-9447-57085013e108"
 					(reference "R1")
 					(unit 1)
@@
 		(instances
 			(project "puck-revA"
-				(path "/5d319f43-1749-4bb5-87ad-5a3caec3474c"
+				(path "/95006bc4-82f3-4f47-9447-57085013e108"
 					(reference "R2")
 					(unit 1)
@@
 		(instances
 			(project "puck-revA"
-				(path "/5d319f43-1749-4bb5-87ad-5a3caec3474c"
+				(path "/95006bc4-82f3-4f47-9447-57085013e108"
 					(reference "R3")
 					(unit 1)
@@
 		(instances
 			(project "puck-revA"
-				(path "/5d319f43-1749-4bb5-87ad-5a3caec3474c"
+				(path "/95006bc4-82f3-4f47-9447-57085013e108"
 					(reference "R4")
 					(unit 1)
@@
 		(instances
 			(project "puck-revA"
-				(path "/5d319f43-1749-4bb5-87ad-5a3caec3474c"
+				(path "/95006bc4-82f3-4f47-9447-57085013e108"
 					(reference "R5")
 					(unit 1)
@@
 		(instances
 			(project "puck-revA"
-				(path "/5d319f43-1749-4bb5-87ad-5a3caec3474c"
+				(path "/95006bc4-82f3-4f47-9447-57085013e108"
 					(reference "R6")
 					(unit 1)
@@
 		(instances
 			(project "puck-revA"
-				(path "/5d319f43-1749-4bb5-87ad-5a3caec3474c"
+				(path "/95006bc4-82f3-4f47-9447-57085013e108"
 					(reference "C1")
 					(unit 1)
@@
 		(instances
 			(project "puck-revA"
-				(path "/5d319f43-1749-4bb5-87ad-5a3caec3474c"
+				(path "/95006bc4-82f3-4f47-9447-57085013e108"
 					(reference "C2")
 					(unit 1)
@@
 		(instances
 			(project "puck-revA"
-				(path "/5d319f43-1749-4bb5-87ad-5a3caec3474c"
+				(path "/95006bc4-82f3-4f47-9447-57085013e108"
 					(reference "C3")
 					(unit 1)
@@
 		(instances
 			(project "puck-revA"
-				(path "/5d319f43-1749-4bb5-87ad-5a3caec3474c"
+				(path "/95006bc4-82f3-4f47-9447-57085013e108"
 					(reference "C4")
 					(unit 1)
@@
 		(instances
 			(project "puck-revA"
-				(path "/5d319f43-1749-4bb5-87ad-5a3caec3474c"
+				(path "/95006bc4-82f3-4f47-9447-57085013e108"
 					(reference "C5")
 					(unit 1)
@@
 		(instances
 			(project "puck-revA"
-				(path "/5d319f43-1749-4bb5-87ad-5a3caec3474c"
+				(path "/95006bc4-82f3-4f47-9447-57085013e108"
 					(reference "C6")
 					(unit 1)
@@
 		(instances
 			(project "puck-revA"
-				(path "/5d319f43-1749-4bb5-87ad-5a3caec3474c"
+				(path "/95006bc4-82f3-4f47-9447-57085013e108"
 					(reference "C7")
 					(unit 1)
@@
 		(instances
 			(project "puck-revA"
-				(path "/5d319f43-1749-4bb5-87ad-5a3caec3474c"
+				(path "/95006bc4-82f3-4f47-9447-57085013e108"
 					(reference "#FLG1")
 					(unit 1)
@@
 		(instances
 			(project "puck-revA"
-				(path "/5d319f43-1749-4bb5-87ad-5a3caec3474c"
+				(path "/95006bc4-82f3-4f47-9447-57085013e108"
 					(reference "#FLG2")
 					(unit 1)

Commit message: hardware(puck): three LEDs will not fit on this board, so there are four
gen_pcb.py places the board from the same PARTS table the schematic comes from,
so the two cannot disagree about what is on it. It places and does not route: the
point is that the geometry the enclosure depends on lives in the file rather than
in somebody's head.

Laying it out turned up a fault no amount of reading would have: THREE LEDS
CANNOT BE PLACED. The module is 18 x 25.5 and lies across the board from the 180
degree edge; the connector holds the 0 degree edge. Between them they block every
ring angle in (129,231) and (328,32), and an equilateral triple always lands one
LED inside one of those. Proven by exhaustive search over every angle and every
ring radius that keeps the emitters 8-10 mm off the diffuser -- and growing the
ring until a symmetric quad fits drops the radial standoff to 6.4 mm, so the cure
is worse than the disease.

Four at {43, 128, 232, 317} keeps the ring at 17 mm and therefore the 8.4 mm
radial standoff the optics were designed around, with a smallest gap of 85
degrees where 90 would be perfect. The two wide gaps land at 0 and 180: the
connector notch, already a hole in the glow, and the antenna side. docs, the
netlist, the schematic and the enclosure's mock all now say four.

The bolt circle moved from 40 mm to 42 for the same kind of reason: at 40 no
equilateral trio of M2 holes clears the LEDs, the module and the connector at
once. At 42, {24, 144, 264} does, with 6.6 mm to the nearest emitter and every
hole more than 30 degrees off the antenna. puck.scad follows it, and has a second
assert now, because bosses and magnets sit on different circles and their angles
alone do not tell you whether they touch.

Three faults in the generator, each caught by a tool rather than by reading:

- The s-expression scanner broke on the first ')' instead of at matching depth,
  so every nested query silently returned nothing.
- Packing used the footprint courtyard, and on ESP3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
Parts:
- added C8: 100n, Capacitor_SMD:C_0603_1608Metric, symbol Device:C
- added D4: SK6812-RGBW, LED_SMD:LED_SK6812_PLCC4_5.0x5.0mm_P3.2mm, symbol LED:WS2812B
- J2: footprint Connector_PinHeader_2.54mm:PinHeader_1x04_P2.54mm_Vertical -> Connector_PinHeader_1.27mm:PinHeader_1x04_P1.27mm_Vertical
- J3: footprint Connector_PinHeader_2.54mm:PinHeader_1x06_P2.54mm_Vertical -> Connector_PinHeader_1.27mm:PinHeader_1x06_P1.27mm_Vertical
Connections:
- net GND: now also C8.2, D4.3 (VSS)
- net VBUS: now also C8.1, D4.1 (VDD)
- net LED_D3_OUT: now reaches D3.2 (DOUT)
- net LED_D3_OUT: now also D4.4 (DIN)

Commit message: hardware(puck): the antenna moves to the roof, and the light becomes a ring
Two of the LEDs were touching the module. That is a symptom: the -1's trace
antenna has to sit at a board edge and drags a 48 x 41 mm keepout with it, and on
a 50 mm disc that blocked a third of every ring radius permanently. It is what
forced four LEDs instead of three, the asymmetric angles, the 42 mm bolt circle
and the crowding.

So the module is an ESP32-S3-WROOM-1U now: same 41 pins, same 16 MB, a U.FL where
the antenna was. A 2.4 GHz flex adheres inside the diffuser roof and the module
moves to the CENTRE of the board, where its castellated pads face outward at
everything they need to reach. The ring goes round it: eleven SK6812-RGBW on
r=17 at 30 deg, the twelfth slot left empty because that is where the connector
is. Cost is one FPC antenna and a U.FL press at assembly. Modular certification
later depends on using an antenna from Espressif's approved list, which is
written down now rather than discovered later. KiCad ships the -1U footprint but
not its symbol -- the -1's is pin-identical, checked pad for pad -- and no -1U
3D model, so it renders as bare pads.

A ring of light AT THE RIM was built, looked at, and rejected. Twenty-one small
LEDs 3.9 mm inside the wall read as a light ring -- a status band, an Echo Dot --
and bead visibly along the bottom of the band where the wall is only 4.6 mm away.
Every board and doc here describes something else: warm, and still; a small,
plain relay object; not a hard point source you can see the die in. That is an
object that glows evenly from within, which you get with fewer emitters further
from the wall, not more of them closer to it. At r=17 they sit 9.0 mm from the
roof and 8.4 mm from the side, deliberately close to equal, so a body whose
orientation nobody can predict glows the same from every angle.

Decoupling went from one cap per LED to four, and that is a decision rather than
a saving: there is nowhere on a single-sided 50 mm board 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
Parts:
- removed C4, C5, C6, C8: 100n, Capacitor_SMD:C_0603_1608Metric, symbol Device:C
- added C101, C102, C103, C104: 100n, Capacitor_SMD:C_0603_1608Metric, symbol Device:C
- added D10, D11, D5, D6, D7, D8, D9: SK6812-RGBW, LED_SMD:LED_SK6812_PLCC4_5.0x5.0mm_P3.2mm, symbol LED:WS2812B
- SW1, SW2, SW3: footprint Button_Switch_SMD:SW_SPST_SKQG_WithoutStem -> Button_Switch_SMD:SW_Push_1P1T-SH_NO_CK_KMR2xxG
- U1: value ESP32-S3-WROOM-1-N16 -> ESP32-S3-WROOM-1U-N16; footprint RF_Module:ESP32-S3-WROOM-1 -> RF_Module:ESP32-S3-WROOM-1U
Connections:
- net GND: now also C101.2, C102.2, C103.2, C104.2, D10.3 (VSS), D11.3 (VSS), D5.3 (VSS), D6.3 (VSS), D7.3 (VSS), D8.3 (VSS), D9.3 (VSS)
- net VBUS: now also C101.1, C102.1, C103.1, C104.1, D10.1 (VDD), D11.1 (VDD), D5.1 (VDD), D6.1 (VDD), D7.1 (VDD), D8.1 (VDD), D9.1 (VDD)
- net LED_D4_OUT: now reaches D4.2 (DOUT)
- net LED_D4_OUT: now also D5.4 (DIN)
- new net LED_D10_OUT: D10.2 (DOUT), D11.4 (DIN)
- new net LED_D5_OUT: D5.2 (DOUT), D6.4 (DIN)
- new net LED_D6_OUT: D6.2 (DOUT), D7.4 (DIN)
- new net LED_D7_OUT: D7.2 (DOUT), D8.4 (DIN)
- new net LED_D8_OUT: D8.2 (DOUT), D9.4 (DIN)
- new net LED_D9_OUT: D10.4 (DIN), D9.2 (DOUT)
