File: hardware/puck-revA/puck-revA.kicad_sch (KiCad schematic)
At the start: 36 parts, among them J1 USB-C 16P, J2 UART, J3 EXP (DNP on the product), SW1 BOOT, SW2 RESET, SW3 USER, U1 ESP32-S3-WROOM-1U-N16, U2 AP2112K-3.3, U3 74AHCT1G125, U4 USBLC6-2SC6, U5 ambient light, DNP

Commit message: Add initial files for Puck hardware revision A
- Created sym-lib-table for project-owned components.
- Added sync-check.json to store synchronization check results.
- Implemented verify_sync.py to compare KiCad-exported nets and components with the PCB layout.
Parts:
- added H1, H2, H3: M2, MountingHole:MountingHole_2.2mm_M2, symbol Mechanical:MountingHole
- added R7: 2k2, Resistor_SMD:R_0402_1005Metric, symbol Device:R
- SW3: value USER -> KMS223G LFG; footprint Button_Switch_SMD:SW_Push_1P1T-SH_NO_CK_KMR2xxG -> Button_Switch_SMD:SW_SPST_CK_KMS2xxG; symbol Switch:SW_Push -> Puck:SW_Push_Shield
Connections:
- net +3V3: now also R7.1
- net GND: now also SW3.SH
- net USER_BTN: now also R7.2
Other:
- moved on the sheet: C1, C101, C102, C103, C104, C2, C3, C7, R1, R2, R3, R4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
