File: hardware/puck-revA/puck-revA.kicad_pcb (KiCad board)
At the start: 2 copper layers, 50 x 50 mm, 39 parts, among them J1 USB-C 16P, J2 UART, J3 EXP (DNP on the product), SW1 BOOT, SW2 RESET, SW3 USER, U1 ESP32-S3-WROOM-1U-N16, U2 AP2112K-3.3, U3 74AHCT1G125, U4 USBLC6-2SC6, U5 ambient light, DNP

Commit message: hardware(puck): the ten shorts were real, and I said they were an artifact
Your DRC report, run in the GUI with the zones actually filled, settled two
things I could not settle headlessly.

GND is genuinely connected. Not one of the 51 unconnected pads is a ground pad,
so the pour on both layers does what route.py --check said it did.

And the ten shorts were REAL. I called them an unfilled-zone artifact on the
strength of a control board -- deleting the F.Cu pour took shorting_items from 10
to 0, so I concluded the pour was the cause. It was not. Deleting the pour just
removed the net that the track was shorting TO. Measured properly, each chain leg
passes 0.42 mm from the centre of the next LED's VSS pad: a pad half-width of
0.75 and a track half-width of 0.125 means 0.46 mm of overlap. The tracks ran
straight through those pads and I shipped it saying they probably did not.

The cause was assuming a path shape. Drop inboard, run round, climb out at the
far end sounds safe and puts the climb through a pad that happens to sit on the
way. So hops are SEARCHED now: generate candidates -- direct, inboard arcs at
five radii, outboard arcs at three -- measure each against every foreign pad, and
take the first that clears 0.95 mm. All ten hops still route, and no track on the
board now passes within 0.95 mm of a pad that is not its own.

Also solid pad connections on the ground pours. J1's ground pads are big enough
that KiCad could only reach them with one thermal spoke where the rule wants two:
six starved_thermal errors, and nothing here is hand-soldered.

Headless DRC now: no shorts, no mask bridges, no starved thermals, no clearance
violations. What it still reports -- unconnected pads and dangling vias -- is the
zone-filling limit, and the signal nets that were never mine to route.

Co-Authored-By: Claude Opus 5 (1M context) <noreply@anthropic.com>
Routing:
- net LED_D8_OUT: track 10.3 -> 5.11 mm
- net LED_D5_OUT: track 10.3 -> 5.11 mm
- net LED_D2_OUT: track 10.3 -> 5.11 mm
- net LED_D7_OUT: track 10.3 -> 5.11 mm
- net LED_D4_OUT: track 10.3 -> 5.11 mm
- net LED_D1_OUT: track 10.3 -> 5.11 mm
- net LED_D10_OUT: track 10.3 -> 5.11 mm
- net LED_D9_OUT: track 10.3 -> 5.11 mm
- net LED_D6_OUT: track 10.3 -> 5.11 mm
- net LED_D3_OUT: track 10.3 -> 5.11 mm
Changed lines of the file:
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@@
 		(priority 0)
 		(hatch edge 0.5)
-		(connect_pads
-			(clearance 0.3)
+		(connect_pads yes
+			(clearance 0)
 		)
 		(min_thickness 0.2)
@@
 		(priority 0)
 		(hatch edge 0.5)
-		(connect_pads
-			(clearance 0.3)
+		(connect_pads yes
+			(clearance 0)
 		)
 		(min_thickness 0.2)
@@
 	(segment
 		(start 112.1118 90.1782)
-		(end 110.5633 91.4339)
+		(end 111.4218 85.117)
 		(width 0.25)
 		(layer "F.Cu")
@@
 	)
 	(segment
-		(start 110.5633 91.4339)
-		(end 108.2799 89.211)
-		(width 0.25)
-		(layer "F.Cu")
-		(net 6)
-	)
-	(segment
-		(start 108.2799 89.211)
-		(end 111.4218 85.117)
-		(width 0.25)
-		(layer "F.Cu")
-		(net 6)
-	)
-	(segment
 		(start 105.5782 85.4382)
-		(end 104.8651 87.3)
+		(end 102.45 81.4)
 		(width 0.25)
 		(layer "F.Cu")
@@
 	)
 	(segment
-		(start 104.8651 87.3)
-		(end 101.7761 86.5165)
-		(width 0.25)
-		(layer "F.Cu")
-		(net 9)
-	)
-	(segment
-		(start 101.7761 86.5165)
-		(end 102.45 81.4)
-		(width 0.25)
-		(layer "F.Cu")
-		(net 9)
-	)
-	(segment
 		(start 97.55 84.6)
-		(end 97.8632 86.5689)
+		(end 92.8218 82.667)
 		(width 0.25)
 		(layer "F.Cu")
@@
 	)
 	(segment
-		(start 97.8632 86.5689)
-		(end 94.7963 87.4349)
-		(width 0.25)
-		(layer "F.Cu")
-		(net 10)
-	)
-	(segment
-		(start 94.7963 87.4349)
-		(end 92.8218 82.667)
-		(width 0.25)
-		(layer "F.Cu")
-		(net 10)
-	)
-	(segment
 		(start 90.1782 87.8882)
-		(end 91.4339 89.4367)
+		(end 85.117 88.5782)
 		(width 0.25)
 		(layer "F.Cu")
@@
 	)
 	(segment
-		(start 91.4339 89.4367)
-		(end 89.211 91.7201)
-		(width 0.25)
-		(layer "F.Cu")
-		(net 11)
-	)
-	(segment
-		(start 89.211 91.7201)
-		(end 85.117 88.5782)
-		(width 0.25)
-		(layer "F.Cu")
-		(net 11)
-	)
-	(segment
 		(start 85.4382 94.4218)
-		(end 87.3 95.1349)
+		(end 81.4 97.55)
 		(width 0.25)
 		(layer "F.Cu")
@@
 	)
 	(segment
-		(start 87.3 95.1349)
-		(end 86.5165 98.2239)
-		(width 0.25)
-		(layer "F.Cu")
-		(net 12)
-	)
-	(segment
-		(start 86.5165 98.2239)
-		(end 81.4 97.55)
-		(width 0.25)
-		(layer "F.Cu")
-		(net 12)
-	)
-	(segment
 		(start 84.6 102.45)
-		(end 86.5689 102.1368)
+		(end 82.667 107.1782)
 		(width 0.25)
 		(layer "F.Cu")
@@
 	)
 	(segment
-		(start 86.5689 102.1368)
-		(end 87.4349 105.2037)
-		(width 0.25)
-		(layer "F.Cu")
-		(net 13)
-	)
-	(segment
-		(start 87.4349 105.2037)
-		(end 82.667 107.1782)
-		(width 0.25)
-		(layer "F.Cu")
-		(net 13)
-	)
-	(segment
 		(start 87.8882 109.8218)
-		(end 89.4367 108.5661)
+		(end 88.5782 114.883)
 		(width 0.25)
 		(layer "F.Cu")
@@
 	)
 	(segment
-		(start 89.4367 108.5661)
-		(end 91.7201 110.789)
-		(width 0.25)
-		(layer "F.Cu")
-		(net 14)
-	)
-	(segment
-		(start 91.7201 110.789)
-		(end 88.5782 114.883)
-		(width 0.25)
-		(layer "F.Cu")
-		(net 14)
-	)
-	(segment
 		(start 94.4218 114.5618)
-		(end 95.1349 112.7)
+		(end 97.55 118.6)
 		(width 0.25)
 		(layer "F.Cu")
@@
 	)
 	(segment
-		(start 95.1349 112.7)
-		(end 98.2239 113.4835)
-		(width 0.25)
-		(layer "F.Cu")
-		(net 15)
-	)
-	(segment
-		(start 98.2239 113.4835)
-		(end 97.55 118.6)
-		(width 0.25)
-		(layer "F.Cu")
-		(net 15)
-	)
-	(segment
 		(start 102.45 115.4)
-		(end 102.1368 113.4311)
+		(end 107.1782 117.333)
 		(width 0.25)
 		(layer "F.Cu")
@@
 	)
 	(segment
-		(start 102.1368 113.4311)
-		(end 105.2037 112.5651)
-		(width 0.25)
-		(layer "F.Cu")
-		(net 7)
-	)
-	(segment
-		(start 105.2037 112.5651)
-		(end 107.1782 117.333)
-		(width 0.25)
-		(layer "F.Cu")
-		(net 7)
-	)
-	(segment
 		(start 109.8218 112.1118)
-		(end 108.5661 110.5633)
-		(width 0.25)
-		(layer "F.Cu")
-		(net 8)
-	)
-	(segment
-		(start 108.5661 110.5633)
-		(end 110.789 108.2799)
-		(width 0.25)
-		(layer "F.Cu")
-		(net 8)
-	)
-	(segment
-		(start 110.789 108.2799)
 		(end 114.883 111.4218)
 		(width 0.25)
