File: hardware/puck-revA/puck-revA.kicad_pcb (KiCad board)
At the start: 2 copper layers, 50 x 50 mm, 39 parts, among them J1 USB-C 16P, J2 UART, J3 EXP (DNP on the product), SW1 BOOT, SW2 RESET, SW3 USER, U1 ESP32-S3-WROOM-1U-N16, U2 AP2112K-3.3, U3 74AHCT1G125, U4 USBLC6-2SC6, U5 ambient light, DNP

Commit message: Add initial files for Puck hardware revision A
- Created sym-lib-table for project-owned components.
- Added sync-check.json to store synchronization check results.
- Implemented verify_sync.py to compare KiCad-exported nets and components with the PCB layout.
Parts:
- added R7: 2k2, Resistor_SMD:R_0402_1005Metric, F.Cu at (89.8, 96.0)
- SW3: value USER -> KMS223G LFG; footprint Button_Switch_SMD:SW_Push_1P1T-SH_NO_CK_KMR2xxG -> Button_Switch_SMD:SW_SPST_CK_KMS2xxG
Connections:
- D11 pad 2: (no net) -> unconnected-(D11-DOUT-Pad2)
- J1 pad A8: (no net) -> unconnected-(J1-SBU1-PadA8)
- J1 pad B8: (no net) -> unconnected-(J1-SBU2-PadB8)
- SW3 pad SH: (no net) -> GND
- U1 pad 15: (no net) -> unconnected-(U1-IO3-Pad15)
- U1 pad 16: (no net) -> unconnected-(U1-IO46-Pad16)
- U1 pad 18: (no net) -> unconnected-(U1-IO10-Pad18)
- U1 pad 19: (no net) -> unconnected-(U1-IO11-Pad19)
- U1 pad 20: (no net) -> unconnected-(U1-IO12-Pad20)
- U1 pad 21: (no net) -> unconnected-(U1-IO13-Pad21)
- U1 pad 22: (no net) -> unconnected-(U1-IO14-Pad22)
- U1 pad 23: (no net) -> unconnected-(U1-IO21-Pad23)
- U1 pad 24: (no net) -> unconnected-(U1-IO47-Pad24)
- U1 pad 25: (no net) -> unconnected-(U1-IO48-Pad25)
- U1 pad 26: (no net) -> unconnected-(U1-IO45-Pad26)
- U1 pad 28: (no net) -> unconnected-(U1-IO35-Pad28)
- U1 pad 29: (no net) -> unconnected-(U1-IO36-Pad29)
- U1 pad 30: (no net) -> unconnected-(U1-IO37-Pad30)
- U1 pad 32: (no net) -> unconnected-(U1-IO39-Pad32)
- U1 pad 33: (no net) -> unconnected-(U1-IO40-Pad33)
- U1 pad 34: (no net) -> unconnected-(U1-IO41-Pad34)
- U1 pad 35: (no net) -> unconnected-(U1-IO42-Pad35)
- U1 pad 38: (no net) -> unconnected-(U1-IO2-Pad38)
- U1 pad 39: (no net) -> unconnected-(U1-IO1-Pad39)
- U1 pad 5: (no net) -> unconnected-(U1-IO5-Pad5)
- U1 pad 6: (no net) -> unconnected-(U1-IO6-Pad6)
- U1 pad 7: (no net) -> unconnected-(U1-IO7-Pad7)
- U1 pad 8: (no net) -> unconnected-(U1-IO15-Pad8)
- U2 pad 4: (no net) -> unconnected-(U2-NC-Pad4)
- U5 pad 2: (no net) -> unconnected-(U5-NC-Pad2)
- U5 pad 5: (no net) -> unconnected-(U5-INT-Pad5)
Routing:
- net GND: track 0.00 -> 6.63 mm, vias 0 -> 10
- net VBUS: track 221.3 -> 216.4 mm
- net +3V3: track 100.5 -> 103.5 mm
- net USB_DP: track 33.1 -> 34.5 mm, vias 4 -> 5
- net USB_DM: track 51.4 -> 52.2 mm, vias 6 -> 5
- net USER_BTN: track 26.9 -> 27.5 mm
- net CC2: vias 1 -> 0
- net CC1: vias 1 -> 0
