File: hardware/archive/puck-revA-before-common-switches-20260926-163743/puck-revA.kicad_pcb (KiCad board)
At the start: 4 copper layers, 50 x 50 mm, 58 parts, among them J1 USB-C 16P, J2 UART, J3 EXP (DNP on the product), Q1 AO3400A, Q2 AO3400A, SW1 KMS221GLFS, SW2 KMS221GLFS, SW3 KMS221GLFS, U1 ESP32-S3-WROOM-1U-N16, U2 TPS62162DSGR, U3 SN74LV1T125DBVR, U4 USBLC6-2SC6, U5 ambient light, DNP, U6 TUSB320IRWBR, U7 TPS22918DBVR, U8 TPS2553DBVR

Commit message: Refactor code structure for improved readability and maintainability
Parts:
- removed R19: 2k2, Resistor_SMD:R_0603_1608Metric
- removed R20: 300, Resistor_SMD:R_0603_1608Metric
- C7: value 10u 16V X5R -> 1u 25V X7R
- R3: value 2k2 -> 10k
- R8: value 887k 1% -> 900k 1%
- SW1: value KMS221GLFS -> BOOT; footprint Button_Switch_SMD:SW_SPST_CK_KMS2xxG -> Button_Switch_SMD:SW_Push_1P1T-SH_NO_CK_KMR2xxG
- SW2: value KMS221GLFS -> RESET; footprint Button_Switch_SMD:SW_SPST_CK_KMS2xxG -> Button_Switch_SMD:SW_Push_1P1T-SH_NO_CK_KMR2xxG
- SW3: value KMS221GLFS -> KMS223G LFG
Connections:
- SW2 pad 1: RESET_SW -> EN
Routing:
- net EN: track 18.2 -> 35.0 mm, vias 2 -> 4
- net RESET_SW: track 15.2 -> 0.00 mm, vias 2 -> 0
- net +3V3: track 175.1 -> 165.2 mm, vias 11 -> 9
- net IO0: track 41.3 -> 36.1 mm
