File: hardware/archive/puck-revA-before-common-switches-20260926-163743/puck-revA.kicad_sch (KiCad schematic)
At the start: 58 parts, among them J1 USB-C 16P, J2 UART, J3 EXP (DNP on the product), Q1 AO3400A, Q2 AO3400A, SW1 KMS221GLFS, SW2 KMS221GLFS, SW3 KMS221GLFS, U1 ESP32-S3-WROOM-1U-N16, U2 TPS62162DSGR, U3 SN74LV1T125DBVR, U4 USBLC6-2SC6, U5 ambient light, DNP, U6 TUSB320IRWBR, U7 TPS22918DBVR, U8 TPS2553DBVR

Commit message: Refactor code structure for improved readability and maintainability
Parts:
- removed R19: 2k2, Resistor_SMD:R_0603_1608Metric, symbol Device:R
- removed R20: 300, Resistor_SMD:R_0603_1608Metric, symbol Device:R
- C7: value 10u 16V X5R -> 1u 25V X7R; LCSC C86275 -> C29936; MPN GRM188R61C106KAALD -> CL10B105KA8NNNC; Manufacturer Murata -> Samsung Electro-Mechanics
- H1, H2, H3: now in the parts list
- R16: LCSC C13187 -> C309561; MPN 0603WAF3242T5E -> RC0603FR-0732K4L; Manufacturer UNI-ROYAL -> YAGEO
- R3: value 2k2 -> 10k; LCSC C4190 -> C25804; MPN 0603WAF2201T5E -> 0603WAF1002T5E
- R8: value 887k 1% -> 900k 1%; LCSC C246015 -> C407504; MPN RC0603FR-07887KL -> 0603WAF9003T5E; Manufacturer YAGEO -> UNI-ROYAL
- SW1: value KMS221GLFS -> BOOT; footprint Button_Switch_SMD:SW_SPST_CK_KMS2xxG -> Button_Switch_SMD:SW_Push_1P1T-SH_NO_CK_KMR2xxG; LCSC C221698 -> (none); MPN KMS221GLFS -> Y78B22114FP; Manufacturer C&K / Littelfuse -> Littelfuse / C&K; Ordering_Alias KMS221G LFS -> KMR221G ULC LFS; Sourcing_Status JLCPCB C221698; side actuated; no pegs; pull-ups revised fo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 -> ULC version required; special procurement or hand assembly;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
- SW2: value KMS221GLFS -> RESET; footprint Button_Switch_SMD:SW_SPST_CK_KMS2xxG -> Button_Switch_SMD:SW_Push_1P1T-SH_NO_CK_KMR2xxG; LCSC C221698 -> (none); MPN KMS221GLFS -> Y78B22114FP; Manufacturer C&K / Littelfuse -> Littelfuse / C&K; Ordering_Alias KMS221G LFS -> KMR221G ULC LFS; Sourcing_Status JLCPCB C221698; side actuated; no pegs; pull-ups revised fo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 -> ULC version required; special procurement or hand assembly;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
- SW3: value KMS221GLFS -> KMS223G LFG; LCSC C221698 -> C35808863; MPN KMS221GLFS -> KMS223GLFG; Ordering_Alias KMS221G LFS -> (none); Sourcing_Status JLCPCB C221698; side actuated; no pegs; pull-ups revised fo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 -> (none)
Connections:
- net RESET_SW is gone; now on net EN: SW2.1
